File: eagle/SOM EVAL BOARD V101.brd (EAGLE design)
At the start: 125 x 90 mm, 170 parts, among them J1 TE 2199230-4, J10 4P-2.0-90D, J11 4P-2.0-90D, J12 CON_62_SMD_HEADER, J2 DCJ0202, J3 SPARK_CON_30X2_SMD, J35 CON_122_SMD_HEADER, J6 SCREW-HOLE-2.6, P1 SPARK_POGOPIN, P2 SPARK_POGOPIN, P3 SPARK_POGOPIN, P4 SPARK_POGOPIN, Q2 IR6401, Q3 IR6401, U1 W5500, U13 MAX1704X, U14 BQ24195L, U2 XC8107SOT25, U3 XC9258A, X1 BU-SMA-G, X3 BU-SMA-G, X4 0046_15TW-882, Y1 25MHz

Commit message: Updated to version 1.0.1 of eval board
Parts:
- added TP1, TP10, TP11, TP12, TP13, TP14, TP15, TP16, TP17, TP18, TP19, TP2, TP20, TP21, TP22, TP23, TP24, TP25, TP26, TP27, TP28, TP29, TP30, TP31, TP32, TP33, TP34, TP35, TP36, TP37, TP38, TP39, TP4, TP40, TP41, TP42, TP43, TP44, TP45, TP46, TP47, TP48, TP49, TP5, TP50, TP51, TP6, TP7, TP8, TP9: TPSB1,27, testpad:B1,27
Connections:
- net /RESET: now also TP33.TP
- net 3V3: now also TP27.TP
- net ADC0: now also TP4.TP
- net ADC1: now also TP5.TP
- net ADC2: now also TP6.TP
- net ADC3: now also TP7.TP
- net ADC4: now also TP9.TP
- net ADC5: now also TP10.TP
- net ADC6: now also TP11.TP
- net ADC7: now also TP12.TP
- net BLUE: now also TP21.TP
- net CS: now also TP38.TP
- net CTS: now also TP36.TP
- net GND: now also TP13.TP, TP42.TP, TP8.TP
- net GPIO0: now also TP45.TP
- net GPIO1: now also TP46.TP
- net GREEN: now also TP20.TP
- net MISO: now also TP39.TP
- net MODE: now also TP32.TP
- net MOSI: now also TP40.TP
- net NC0: now also TP28.TP
- net NC1: now also TP29.TP
- net NC11: now also TP14.TP
- net NC12: now also TP15.TP
- net NC13: now also TP16.TP
- net NC14: now also TP17.TP
- net NC15: now also TP18.TP
- net NC2: now also TP43.TP
- net NC3: now also TP44.TP
- net NFC1: now also TP1.TP
- net NFC2: now also TP2.TP
- net PWM0: now also TP47.TP
- net PWM1: now also TP48.TP
- net PWM2: now also TP49.TP
- net PWM3: now also TP50.TP
- net RED: now also TP19.TP
- net RTS: now also TP37.TP
- net RX: now also TP35.TP
- net SCK: now also TP41.TP
- net SCL: now also TP30.TP
- net SDA: now also TP31.TP
- net SOM5: now also TP22.TP
- net SOM6: now also TP23.TP
- net SOM7: now also TP24.TP
- net SOM8: now also TP25.TP
- net SOM9: now also TP26.TP
- net TX: now also TP34.TP
- net VCC: now also TP51.TP
Routing:
- net GND: track 175.4 -> 190.0 mm, vias 773 -> 777
- net BLUE: track 78.2 -> 87.2 mm
- net NC12: track 17.4 -> 22.3 mm, vias 0 -> 1
- net SOM8: track 31.3 -> 36.1 mm, vias 0 -> 1
- net ADC1: track 76.8 -> 81.6 mm, vias 1 -> 2
- net GREEN: track 81.9 -> 86.7 mm
- net ADC4: track 25.4 -> 30.1 mm, vias 0 -> 1
- net ADC3: track 28.2 -> 33.0 mm, vias 0 -> 1
- net SOM6: track 29.9 -> 34.6 mm, vias 0 -> 1
- net ADC2: track 73.6 -> 78.3 mm, vias 1 -> 2
- net SOM7: track 31.2 -> 35.9 mm, vias 0 -> 1
- net NC13: track 17.5 -> 22.2 mm, vias 0 -> 1
- net NC11: track 18.7 -> 23.4 mm, vias 0 -> 1
- net ADC5: track 25.1 -> 29.8 mm, vias 0 -> 1
- net ADC7: track 108.9 -> 113.6 mm, vias 2 -> 3
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Other:
- board text added: "SOM EVAL BOARD V101"
- board text added: "SoM5"
- board text added: "SoM6"
- board text added: "SoM7"
- board text added: "SoM8"
- board text added: "SoM9"
- board text removed: "SOM EVAL BOARD V1.00"
- board text removed: "SOM5"
- board text removed: "SOM6"
- board text removed: "SOM7"
- board text removed: "SOM8"
- board text removed: "SOM9"
