File: eagle/SOM EVAL BOARD V101.sch (EAGLE design)
At the start: 170 parts, among them J1 TE 2199230-4, J10 4P-2.0-90D, J11 4P-2.0-90D, J12 CON_62_SMD_HEADER, J2 DCJ0202, J3 SPARK_CON_30X2_SMD, J35 CON_122_SMD_HEADER, J6 SCREW-HOLE-2.6, P1 SPARK_POGOPIN, P2 SPARK_POGOPIN, P3 SPARK_POGOPIN, P4 SPARK_POGOPIN, Q2 IR6401, Q3 IR6401, U1 W5500, U13 MAX1704X, U14 BQ24195L, U2 XC8107SOT25, U3 XC9258A, X1 BU-SMA-G, X3 BU-SMA-G, X4 0046_15TW-882, Y1 25MHz

Commit message: Updated to version 1.0.1 of eval board
Parts:
- added TP1, TP10, TP11, TP12, TP13, TP14, TP15, TP16, TP17, TP18, TP19, TP2, TP20, TP21, TP22, TP23, TP24, TP25, TP26, TP27, TP28, TP29, TP30, TP31, TP32, TP33, TP34, TP35, TP36, TP37, TP38, TP39, TP4, TP40, TP41, TP42, TP43, TP44, TP45, TP46, TP47, TP48, TP49, TP5, TP50, TP51, TP6, TP7, TP8, TP9: TPSB1,27, testpad:TPSB1,27
Connections:
- net /RESET: now also TP33.PP
- net 3V3: now also TP27.PP
- net ADC0: now also TP4.PP
- net ADC1: now also TP5.PP
- net ADC2: now also TP6.PP
- net ADC3: now also TP7.PP
- net ADC4: now also TP9.PP
- net ADC5: now also TP10.PP
- net ADC6: now also TP11.PP
- net ADC7: now also TP12.PP
- net BLUE: now also TP21.PP
- net CS: now also TP38.PP
- net CTS: now also TP36.PP
- net GND: now also TP13.PP, TP42.PP, TP8.PP
- net GPIO0: now also TP45.PP
- net GPIO1: now also TP46.PP
- net GREEN: now also TP20.PP
- net MISO: now also TP39.PP
- net MODE: now also TP32.PP
- net MOSI: now also TP40.PP
- net NC0: now also TP28.PP
- net NC1: now also TP29.PP
- net NC11: now also TP14.PP
- net NC12: now also TP15.PP
- net NC13: now also TP16.PP
- net NC14: now also TP17.PP
- net NC15: now also TP18.PP
- net NC2: now also TP43.PP
- net NC3: now also TP44.PP
- net NFC1: now also TP1.PP
- net NFC2: now also TP2.PP
- net PWM0: now also TP47.PP
- net PWM1: now also TP48.PP
- net PWM2: now also TP49.PP
- net PWM3: now also TP50.PP
- net RED: now also TP19.PP
- net RTS: now also TP37.PP
- net RX: now also TP35.PP
- net SCK: now also TP41.PP
- net SCL: now also TP30.PP
- net SDA: now also TP31.PP
- net SOM5: now also TP22.PP
- net SOM6: now also TP23.PP
- net SOM7: now also TP24.PP
- net SOM8: now also TP25.PP
- net SOM9: now also TP26.PP
- net TX: now also TP34.PP
- net VCC: now also TP51.PP
